Commit message: ros2 control added

File: ur5_description/urdf/ur5_joints_links.xacro (robot description, xacro)
@@ -2,5 +2,5 @@
 <robot xmlns:xacro="http://ros.org/wiki/xacro">
   <xacro:macro name="ur5_joints_links">
-    <!-- links: main serial chain -->
+    <!-- links main serial chain -->
     <link name="world" />
     <link name="base_link">
@@ -8,14 +8,14 @@
         <origin rpy="0 0 3.141592653589793" xyz="0 0 0" />
         <geometry>
-          <mesh filename="package://ur5_description/meshes/visual/base.dae" />
-        </geometry>
-        <material name="LightGrey">
-          <color rgba="0.7 0.7 0.7 1.0" />
-        </material>
-      </visual>
-      <collision>
-        <origin rpy="0 0 3.141592653589793" xyz="0 0 0" />
-        <geometry>
-          <mesh filename="package://ur5_description/meshes/collision/base.stl" />
+          <mesh filename="package://ur5_description/meshes/base.dae" />
+        </geometry>
+        <material name="LightGrey">
+          <color rgba="0.7 0.7 0.7 1.0" />
+        </material>
+      </visual>
+      <collision>
+        <origin rpy="0 0 3.141592653589793" xyz="0 0 0" />
+        <geometry>
+          <mesh filename="package://ur5_description/meshes/base.dae" />
         </geometry>
       </collision>
@@ -30,14 +30,14 @@
         <origin rpy="0 0 3.141592653589793" xyz="0 0 0" />
         <geometry>
-          <mesh filename="package://ur5_description/meshes/visual/shoulder.dae" />
-        </geometry>
-        <material name="LightGrey">
-          <color rgba="0.7 0.7 0.7 1.0" />
-        </material>
-      </visual>
-      <collision>
-        <origin rpy="0 0 3.141592653589793" xyz="0 0 0" />
-        <geometry>
-          <mesh filename="package://ur5_description/meshes/collision/shoulder.stl" />
+          <mesh filename="package://ur5_description/meshes/shoulder.dae" />
+        </geometry>
+        <material name="LightGrey">
+          <color rgba="0.7 0.7 0.7 1.0" />
+        </material>
+      </visual>
+      <collision>
+        <origin rpy="0 0 3.141592653589793" xyz="0 0 0" />
+        <geometry>
+          <mesh filename="package://ur5_description/meshes/shoulder.dae" />
         </geometry>
       </collision>
@@ -53,5 +53,5 @@
         <origin rpy="1.5707963267948966 0 -1.5707963267948966" xyz="0 0 0.138" />
         <geometry>
-          <mesh filename="package://ur5_description/meshes/visual/upperarm.dae" />
+          <mesh filename="package://ur5_description/meshes/upperarm.dae" />
         </geometry>
         <material name="LightGrey">
@@ -62,5 +62,5 @@
         <origin rpy="1.5707963267948966 0 -1.5707963267948966" xyz="0 0 0.138" />
         <geometry>
-          <mesh filename="package://ur5_description/meshes/collision/upperarm.stl" />
+          <mesh filename="package://ur5_description/meshes/upperarm.dae" />
         </geometry>
       </collision>
@@ -76,5 +76,5 @@
         <origin rpy="1.5707963267948966 0 -1.5707963267948966" xyz="0 0 0.007" />
         <geometry>
-          <mesh filename="package://ur5_description/meshes/visual/forearm.dae" />
+          <mesh filename="package://ur5_description/meshes/forearm.dae" />
         </geometry>
         <material name="LightGrey">
@@ -85,5 +85,5 @@
         <origin rpy="1.5707963267948966 0 -1.5707963267948966" xyz="0 0 0.007" />
         <geometry>
-          <mesh filename="package://ur5_description/meshes/collision/forearm.stl" />
+          <mesh filename="package://ur5_description/meshes/forearm.dae" />
         </geometry>
       </collision>
@@ -99,5 +99,5 @@
         <origin rpy="1.5707963267948966 0 0" xyz="0 0 -0.127" />
         <geometry>
-          <mesh filename="package://ur5_description/meshes/visual/wrist1.dae" />
+          <mesh filename="package://ur5_description/meshes/wrist1.dae" />
         </geometry>
         <material name="LightGrey">
@@ -108,5 +108,5 @@
         <origin rpy="1.5707963267948966 0 0" xyz="0 0 -0.127" />
         <geometry>
-          <mesh filename="package://ur5_description/meshes/collision/wrist1.stl" />
+          <mesh filename="package://ur5_description/meshes/wrist1.dae" />
         </geometry>
       </collision>
@@ -122,5 +122,5 @@
         <origin rpy="0 0 0" xyz="0 0 -0.0997" />
         <geometry>
-          <mesh filename="package://ur5_description/meshes/visual/wrist2.dae" />
+          <mesh filename="package://ur5_description/meshes/wrist2.dae" />
         </geometry>
         <material name="LightGrey">
@@ -131,5 +131,5 @@
         <origin rpy="0 0 0" xyz="0 0 -0.0997" />
         <geometry>
-          <mesh filename="package://ur5_description/meshes/collision/wrist2.stl" />
+          <mesh filename="package://ur5_description/meshes/wrist2.dae" />
         </geometry>
       </collision>
@@ -145,5 +145,5 @@
         <origin rpy="1.5707963267948966 0 0" xyz="0 0 -0.0989" />
         <geometry>
-          <mesh filename="package://ur5_description/meshes/visual/wrist3.dae" />
+          <mesh filename="package://ur5_description/meshes/wrist3.dae" />
         </geometry>
         <material name="LightGrey">
@@ -154,5 +154,5 @@
         <origin rpy="1.5707963267948966 0 0" xyz="0 0 -0.0989" />
         <geometry>
-          <mesh filename="package://ur5_description/meshes/collision/wrist3.stl" />
+          <mesh filename="package://ur5_description/meshes/wrist3.dae" />
         </geometry>
       </collision>
@@ -164,5 +164,5 @@
       </inertial>
     </link>
-    <!-- joints: main serial chain -->
+    <!-- joints main serial chain -->
     <joint name="base_fixed_joint" type="fixed">
       <parent link="world"/>
@@ -170,5 +170,5 @@
       <origin xyz="0 0 0" rpy="0 0 0"/>
     </joint>
-    <joint name="joint1" type="revolute">
+    <joint name="joint_1" type="revolute">
       <parent link="base_link" />
       <child link="shoulder_link" />
@@ -178,5 +178,5 @@
         velocity="3.141592653589793" />
     </joint>
-    <joint name="joint2" type="revolute">
+    <joint name="joint_2" type="revolute">
       <parent link="shoulder_link" />
       <child link="upper_arm_link" />
@@ -186,5 +186,5 @@
         velocity="3.141592653589793" />
     </joint>
-    <joint name="joint3" type="revolute">
+    <joint name="joint_3" type="revolute">
       <parent link="upper_arm_link" />
       <child link="forearm_link" />
@@ -194,5 +194,5 @@
         velocity="3.141592653589793" />
     </joint>
-    <joint name="joint4" type="revolute">
+    <joint name="joint_4" type="revolute">
       <parent link="forearm_link" />
       <child link="wrist_1_link" />
@@ -202,5 +202,5 @@
         velocity="3.141592653589793" />
     </joint>
-    <joint name="joint5" type="revolute">
+    <joint name="joint_5" type="revolute">
       <parent link="wrist_1_link" />
       <child link="wrist_2_link" />
@@ -210,5 +210,5 @@
         velocity="3.141592653589793" />
     </joint>
-    <joint name="joint6" type="revolute">
+    <joint name="joint_6" type="revolute">
       <parent link="wrist_2_link" />
       <child link="wrist_3_link" />

File: ur5_description/urdf/ur5_transmissions.xacro (robot description, xacro)
@@ -5,5 +5,5 @@
         <plugin>transmission_interface/SimpleTransmission</plugin>
         <actuator name="joint1_motor" role="joint1_motor" />
-        <joint name="joint1" role="joint1">
+        <joint name="joint_1" role="joint_1">
             <mechanical_reduction>1.0</mechanical_reduction>
         </joint>
@@ -12,5 +12,5 @@
         <plugin>transmission_interface/SimpleTransmission</plugin>
         <actuator name="joint2_motor" role="joint2_motor" />
-        <joint name="joint2" role="joint2">
+        <joint name="joint_2" role="joint_2">
             <mechanical_reduction>1.0</mechanical_reduction>
         </joint>
@@ -19,5 +19,5 @@
         <plugin>transmission_interface/SimpleTransmission</plugin>
         <actuator name="joint3_motor" role="joint3_motor" />
-        <joint name="joint3" role="joint3">
+        <joint name="joint_3" role="joint_3">
             <mechanical_reduction>1.0</mechanical_reduction>
         </joint>
@@ -26,5 +26,5 @@
         <plugin>transmission_interface/SimpleTransmission</plugin>
         <actuator name="joint4_motor" role="joint4_motor" />
-        <joint name="joint4" role="joint4">
+        <joint name="joint_4" role="joint_4">
             <mechanical_reduction>1.0</mechanical_reduction>
         </joint>
@@ -33,5 +33,5 @@
         <plugin>transmission_interface/SimpleTransmission</plugin>
         <actuator name="joint5_motor" role="joint5_motor" />
-        <joint name="joint5" role="joint5">
+        <joint name="joint_5" role="joint_5">
             <mechanical_reduction>1.0</mechanical_reduction>
         </joint>
@@ -40,5 +40,5 @@
         <plugin>transmission_interface/SimpleTransmission</plugin>
         <actuator name="joint6_motor" role="joint6_motor" />
-        <joint name="joint6" role="joint6">
+        <joint name="joint_6" role="joint_6">
             <mechanical_reduction>1.0</mechanical_reduction>
         </joint>

File: ur5_description/urdf/ur5_urdf.xacro (robot description, xacro)
@@ -10,5 +10,5 @@
   <xacro:ur5_transmissions />
   <!-- include ur5 ros2_control description -->
-  <xacro:include filename="$(find ur5_description)/urdf/ur5.ros2_control.xacro" />
+  <xacro:include filename="$(find ur5_description)/urdf/ur5_ros2_control.xacro" />
   <xacro:ur5_ros2_control />
 </robot>
